File: sam3u_breakout.sch (EAGLE design)
At the start: 26 parts, among them IC1 SAM3U_LQFP100

Commit message: Route board
Parts:
- removed C13, C16: (no value), nonolith:CAP_CERAMIC0402
- removed JP1, JP2: (no value), adafruit:PINHD-2X20
- added U$10, U$11, U$12, U$13: M191X19_NO_SILK, SparkFun-Connectors:M191X19_NO_SILK
- added U$14: VREF, nonolith:VREF
Connections:
- removed net N$3: C14.P$2, C15.P$2, C16.P$2, C5.P$2, C6.P$2, C7.P$2, C8.P$2, IC1.VDDCORE, IC1.VDDCORE@1, IC1.VDDCORE@2, IC1.VDDCORE@3, IC1.VDDCORE@4, IC1.VDDOUT, IC1.VDDPLL
- new net 1.8V: C14.P$2, C15.P$2, C5.P$2, C6.P$2, C7.P$2, C8.P$2, IC1.VDDCORE, IC1.VDDCORE@1, IC1.VDDCORE@2, IC1.VDDCORE@3, IC1.VDDCORE@4, IC1.VDDOUT, IC1.VDDPLL
- new net ADVREF: IC1.AD12BVREF, IC1.ADVREF, U$12.9, U$14.VO
- new net ERASE: IC1.ERASE, U$11.12
- new net FWUP: IC1.FWUP, U$10.12
- new net JTAGSEL: IC1.JTAGSEL, U$11.11
- new net N$17: IC1.XOUT32
- new net N$18: IC1.XIN32
- new net NRST: IC1.NRST, U$10.7
- new net NRSTB: IC1.NRSTB, U$10.11
- new net PA0: IC1.PA0, U$11.19
- new net PA1: IC1.PA1, U$10.18
- new net PA10: IC1.PA10, U$11.14
- new net PA11: IC1.PA11, U$10.13
- new net PA12: IC1.PA12, U$11.13
- new net PA13: IC1.PA13, U$13.12
- new net PA14: IC1.PA14, U$12.12
- new net PA15: IC1.PA15, U$13.13
- new net PA16: IC1.PA16, U$12.13
- new net PA17: IC1.PA17, U$13.14
- new net PA18: IC1.PA18, U$12.15
- new net PA19: IC1.PA19, U$13.16
- new net PA2: IC1.PA2, U$11.18
- new net PA20: IC1.PA20, U$12.16
- new net PA21: IC1.PA21, U$13.17
- new net PA22: IC1.PA22, U$13.10
- new net PA23: IC1.PA23, U$12.17
- new net PA24: IC1.PA24, U$13.18
- new net PA25: IC1.PA25, U$12.18
- new net PA26: IC1.PA26, U$13.19
- new net PA27: IC1.PA27, U$12.6
- new net PA28: IC1.PA28, U$13.2
- new net PA29: IC1.PA29, U$12.2
- new net PA3: IC1.PA3, U$10.17
- new net PA30: IC1.PA30, U$12.10
- new net PA31: IC1.PA31, U$13.3
- new net PA4: IC1.PA4, U$11.17
- new net PA5: IC1.PA5, U$10.16
- new net PA6: IC1.PA6, U$11.16
- new net PA7: IC1.PA7, U$10.15
- new net PA8: IC1.PA8, U$11.15
- new net PA9: IC1.PA9, U$10.14
- new net PB0: IC1.PB0, U$12.3
- new net PB1: IC1.PB1, U$13.4
- new net PB10: IC1.PB10, U$10.2
- new net PB11: IC1.PB11, U$13.5
- new net PB12: IC1.PB12, U$12.5
- new net PB13: IC1.PB13, U$13.6
- new net PB14: IC1.PB14, U$11.3
- new net PB15: IC1.PB15, U$13.15
- new net PB16: IC1.PB16, U$12.14
- new net PB17: IC1.PB17, U$10.3
- new net PB18: IC1.PB18, U$11.4
- new net PB19: IC1.PB19, U$10.4
- new net PB2: IC1.PB2, U$12.4
- new net PB20: IC1.PB20, U$11.5
- new net PB21: IC1.PB21, U$10.5
- new net PB22: IC1.PB22, U$11.6
- new net PB23: IC1.PB23, U$10.6
- new net PB24: IC1.PB24, U$11.7
- new net PB3: IC1.PB3, U$13.11
- new net PB4: IC1.PB4, U$12.11
- new net PB5: IC1.PB5, U$13.7
- new net PB6: IC1.PB6, U$12.7
- new net PB7: IC1.PB7, U$13.8
- new net PB8: IC1.PB8, U$12.8
- new net PB9: IC1.PB9, U$11.2
- new net TCK: IC1.TCK, U$11.8
- new net TDI: IC1.TDI, U$10.9
- new net TDO: IC1.TDO, U$11.9
- new net TMS: IC1.TMS, U$10.8
- new net TST: IC1.TST
- net 3.3V: now also U$11.10, U$13.1, U$14.VIN; no longer C13.P$2
- net 5V: now also U$11.1
- net GND: now also U$10.1, U$10.10, U$10.19, U$12.1, U$12.19, U$13.9, U$14.GND; no longer C13.P$1, C16.P$1

Commit message: Labels
Parts:
- renumbered U$10 to HEADER1, U$11 to HEADER2, U$12 to HEADER4, U$13 to HEADER3

Commit message: s/miniusb/microusb/
Parts:
- CN1: device nonolith:USBMINIB -> nonolith:USBMICROB
Changed lines of the file:
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@@
 <?xml version="1.0" encoding="utf-8"?>
 <!DOCTYPE eagle SYSTEM "eagle.dtd">
-<eagle version="6.1">
+<eagle version="6.3">
 <drawing>
 <settings>
@@
 <part name="C8" library="nonolith" deviceset="CAP_CERAMIC" device="0402"/>
 <part name="U$3" library="nonolith" deviceset="GND" device=""/>
-<part name="CN1" library="nonolith" deviceset="USB" device="MINIB"/>
+<part name="CN1" library="nonolith" deviceset="USB" device="MICROB"/>
 <part name="R1" library="nonolith" deviceset="RESISTOR" device="0603" value="39"/>
 <part name="R2" library="nonolith" deviceset="RESISTOR" device="0603" value="39"/>
